File: Radar1.kicad_sch (KiCad schematic)
At the start: 33 parts, among them J1 USB4215-03-A, J2 Barrel_Jack, U1 BGT24LTR11N16, U10 93LC56B-I/SN, U11 445I23D12M00000, U12 AMM-8211PSM, U2 ADF4159WCCPZ, U3 OPA1656ID, U4 TPS7A2033PDBVR, U5 TPS7A2018PDBVR, U6 TPS7A4700RGWT, U7 FT2232HL-REEL, U8 ADS8353IPW, U9 ADP5600ACPZ-R7, Y1 ECS-TXO-2520MV-500-AN-TR

Commit message: Wire signal chain: PLL, IF, RF, USB/SPI, bias networks (WIP checkpoint)
Connected nets 8 -> 58; added 43 components. All connections verified by
kicad-cli netlist export with regression checks; ERC clean of real shorts.

- Regulators: TPS7A4700 programmed to 5.0V + NR cap
- Reference: TCXO -> ADF4159 REFIN, enable tied high
- PLL: 3rd-order loop filter (CP->V_TUNE), DIV_OUT->RFINA feedback, RSET,
  SDVDD decouple, BGT24 R_TUNE/V_PTAT/VCC_PTAT
- TX: BGT24 TX -> AMM-8211 RF_IN, AMM drain bias + decoupling
- IF/RX: placed missing OPA1656 power unit, fixed mis-wired inputs, added
  mid-rail VREF + non-inverting gain (x11) on I/Q, OUT -> ADS8353, ref caps
- Digital: SPI bus (FT2232 <-> ADF4159 <-> ADS8353), USB D+/-, EEPROM,
  FT2232 crystal + load caps
- Negative bias: ADP5600 charge-pump network -> -VGG (AMM gate)
- Fixes: USB shield/GND, ADP5600 EPAD, SDO_A/B short, NC flags, stray labels

Placeholder values needing review: loop filter, IF gain, ADP5600 FB/config,
AMM drain rail (3V3 marginal vs 3.0V spec). Still open: antenna connectors
(RX/RF_OUT), C1-C3 intent, USB VBUS source, new-part footprints.

Co-Authored-By: Claude Opus 4.8 <noreply@anthropic.com>
Parts:
- added C17: 1nF, symbol Device:C_Small_US
- added C18, C33: 10nF, symbol Device:C_Small_US
- added C19: 470pF, symbol Device:C_Small_US
- added C20, C21: 100pF, symbol Device:C_Small_US
- added C22, C23, C30, C31, C32, C35, C36, C37, C42: 100nF, symbol Device:C_Small_US
- added C24, C26, C34, C38, C39, C41: 1uF, symbol Device:C_Small_US
- added C25, C27, C40: 10uF, symbol Device:C_Small_US
- added C28, C29: 18pF, symbol Device:C_Small_US
- added R10, R13, R16, R3, R6, R9: 10k, symbol Device:R_Small_US
- added R11, R14, R17, R19: 100k, symbol Device:R_Small_US
- added R12, R15: 1k, symbol Device:R_Small_US
- added R18: 33k, symbol Device:R_Small_US
- added R4: 2.2k, symbol Device:R_Small_US
- added R5, R7, R8: 5.1k, symbol Device:R_Small_US
- added unit 3 of U3
Connections:
- net +3V3_RF: now also U1.16 (VCC_PTAT), U10.8 (VCC), U12.14 (Vd3), U12.15 (Vd2), U12.16 (Vd1), U2.7 (AVDD), U2.8 (AVDD), Y1.1 (TRI-STATE), C30.1, C31.1, C32.1, R19.1
- net +5V: now also U6.3 (SENSE_FB), R9.1, U3.8 (V+); no longer U3.3 (IN+), U3.5 (IN+)
- net +VIN: now also U9.2 (EN)
- net -VGG: now also U9.11 (CPOUT), U9.8 (CPOUT), C40.1, C42.1, R17.1
- net GND: now also J1.13 (GND), J1.14 (GND), J1.15 (GND), J1.16 (GND), J1.B1/A12 (GND), U10.5 (VSS), U6.10 (0P4V), U6.6 (3P2V), U9.14 (SEL2), U9.15 (SEL1), U9.17 (EPAD), U9.3 (SYNC), U9.4 (FREQ), C17.2, C18.2, C19.2, C21.2, C22.2, C23.2, C24.2, C25.2, C26.2, C27.2, C28.2, C29.2, C30.2, C31.2, C32.2, C33.2, C34.2, C35.2, C40.2, C41.2, C42.2, R10.2, R18.2, R5.2, R6.2, R7.2, R8.2, U3.4 (V-); no longer U3.2 (IN-), U3.6 (IN-)
- net IFA_OUT: now reaches U8.1 (AINP_A)
- net IFA_OUT: now also U3.1 (OUT), R13.2
- net SPI_MOSI: now reaches U8.10 (SDI)
- net SPI_MOSI: now also U2.15 (DATA), U7.17 (ADBUS1)
- net CS_ADC: now reaches U8.11 (*CS)
- net CS_ADC: now also U7.21 (ADBUS4)
- net SPI_SCK: now reaches U8.12 (SCLK)
- net SPI_SCK: now also U2.14 (CLK), U7.16 (ADBUS0)
- net SPI_MISO: now reaches U8.13 (SDO_A)
- net SPI_MISO: now also U7.18 (ADBUS2)
- net VREF: now reaches U8.2 (AINM_A)
- net VREF: now also U8.7 (AINM_B), C34.1, C35.1, R10.1, R11.2, R12.2, R14.2, R15.2, R9.2
- net REFA_N: now reaches U8.3 (REFIO_A)
- net REFA_N: now also C24.1, C25.1
- net REFB_N: now reaches U8.6 (REFIO_B)
- net REFB_N: now also C26.1, C27.1
- net IFB_OUT: now reaches U8.8 (AINP_B)
- net IFB_OUT: now also U3.7 (OUT), R16.2
- net REF_CLK: now reaches Y1.3 (OUTPUT)
- net REF_CLK: now also U2.9 (REFIN)
- net CS_PLL: now reaches U7.19 (ADBUS3)
- net CS_PLL: now also U2.16 (LE)
- net OSC_I: now reaches U7.2 (OSCI)
- net OSC_I: now also U11.1, C28.1
- net ADF_CE: now reaches U7.22 (ADBUS5)
- net ADF_CE: now also U2.13 (CE)
- net ADF_MUXOUT: now reaches U7.23 (ADBUS6)
- net ADF_MUXOUT: now also U2.17 (MUXOUT)
- net ADF_TXDATA: now reaches U7.24 (ADBUS7)
- net ADF_TXDATA: now also U2.12 (TXDATA)
- net BGT_TXEN: now reaches U7.26 (ACBUS0)
- net BGT_TXEN: now also U1.5 (TX_EN)
- net OSC_O: now reaches U7.3 (OSCO)
- net OSC_O: now also U11.2, C29.1
- net EE_DATA: now reaches U7.61 (EEDATA)
- net EE_DATA: now also U10.3 (DI), U10.4 (DO)
- net EE_CLK: now reaches U7.62 (EECLK)
- net EE_CLK: now also U10.2 (CLK)
- net EE_CS: now reaches U7.63 (EECS)
- net EE_CS: now also U10.1 (CS)
- net USB_DM: now reaches U7.7 (DM)
- net USB_DM: now also J1.A7 (DN1), J1.B7 (DN2)
- net USB_DP: now reaches U7.8 (DP)
- net USB_DP: now also J1.A6 (DP1), J1.B6 (DP2)
- net RF_TX: now reaches U12.2 (RF_IN)
- net RF_TX: now also U1.11 (TX)
- net U9C2P: now reaches U9.10 (C2+)
- net U9C2P: now also C39.1
- net U9C1P: now reaches U9.12 (C1+)
- net U9C1P: now also C38.1
- net U9C1N: now reaches U9.13 (C1-)
- net U9C1N: now also C38.2
- net U9PG: now reaches U9.5 (PGOOD)
- net U9PG: now also R19.2
- net U9FB: now reaches U9.6 (FB)
- net U9FB: now also R17.2, R18.1
- net U9LDO: now reaches U9.7 (LDO_OUT)
- net U9LDO: now also C41.1
- net U9C2N: now reaches U9.9 (C2-)
- net U9C2N: now also C39.2
- net NR_N: now reaches U6.14 (NR)
- net NR_N: now also C33.1
- net CC1_N: now reaches J1.A5 (CC1)
- net CC1_N: now also R7.1
- net CC2_N: now reaches J1.B5 (CC2)
- net CC2_N: now also R8.1
- net SDVDD_N: now reaches U2.18 (SDVDD)
- net SDVDD_N: now also C22.1
- net RSET_N: now reaches U2.23 (RSET)
- net RSET_N: now also R5.1
- net LF_A: now reaches U2.24 (CP)
- net LF_A: now also C17.1, R3.1
- net RFINB_N: now reaches U2.4 (RFINB)
- net RFINB_N: now also C21.1
- net RFINA_N: now reaches U2.5 (RFINA)
- net RFINA_N: now also C20.2
- net RTUNE_N: now reaches U1.13 (R_TUNE)
- net RTUNE_N: now also R6.1
- net LF_C: now reaches U1.14 (V_TUNE)
- net LF_C: now also C19.1, R4.2
- net VPTAT_N: now reaches U1.15 (V_PTAT)
- net VPTAT_N: now also C23.1
- net IFQ_IN: now reaches U1.6 (IFQ)
- net IFQ_IN: now also C37.1
- net IFI_IN: now reaches U1.7 (IFI)
- net IFI_IN: now also C36.1
- net DIVO: now reaches U1.8 (DIV_OUT)
- net DIVO: now also C20.1
- new net IFA_INP: C36.2, R11.1, U3.3 (IN+)
- new net IFA_INV: R12.1, R13.1, U3.2 (IN-)
- new net IFB_INP: C37.2, R14.1, U3.5 (IN+)
- new net IFB_INV: R15.1, R16.1, U3.6 (IN-)
- new net LF_B: C18.1, R3.2, R4.1
- no-connect marks 0 -> 19
