File: Radar1.kicad_sch (KiCad schematic)
At the start: 98 parts, among them J1 USB4215-03-A, J2 Barrel_Jack, J3 SMA-2.92mm-EndLaunch, J4 SMA-2.92mm-EndLaunch, U1 BGT24LTR11N16, U10 93LC56B-I/SN, U11 445I23D12M00000, U12 AMM-8211PSM, U13 TPS7A4700RGWT, U14 TPS7A2033PDBVR, U15 TPD2E009DBZR, U16 REF5025AID, U2 ADF4159WCCPZ, U3 OPA1656ID, U4 TPS7A2033PDBVR, U5 TPS7A2018PDBVR, U6 TPS7A4700RGWT, U7 FT2232HL-REEL, U8 ADS8353IPW, U9 ADP5600ACPZ-R7, Y1 ECS-TXO-2520MV-500-AN-TR

Commit message: Rev-D: move FT2232 ADBUS bank, ADS8353 DVDD, MUXOUT pull-up to 1.8V domain
Fixes ADF4159 digital abs-max violation (3.3V into DVDD+0.3V=2.1V pins).
Netlist-regression verified; ERC unchanged.

Co-Authored-By: Claude Fable 5 <noreply@anthropic.com>
Parts:
- added C55: 100nF, Capacitor_SMD:C_0603_1608Metric, symbol Device:C_Small_US
Connections:
- net +1V8: now also C12.1, R22.2, U7.20 (VCCIO-1), U8.9 (DVDD), C55.1
- net +3V3_DIG: no longer R22.2, U7.20 (VCCIO-1)
- net +3V3_RF: no longer C12.1, U8.9 (DVDD)
- net GND: now also C55.2
Changed lines of the file:
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@@
 		)
 	)
-	(global_label "+3V3_DIG"
+	(global_label "+1V8"
 		(shape input)
 		(at 217.17 34.29 0)
@@
 		)
 	)
-	(global_label "+3V3_DIG"
+	(global_label "+1V8"
 		(shape input)
 		(at 373.38 227.33 90)
@@
 		)
 	)
-	(global_label "+3V3_RF"
+	(global_label "+1V8"
 		(shape input)
 		(at 100.33 185.42 270)
@@
 		)
 	)
-	(sheet_instances
+(symbol
+		(lib_id "Device:C_Small_US")
+		(at 381 222.25 90)
+		(unit 1)
+		(exclude_from_sim no)
+		(in_bom yes)
+		(on_board yes)
+		(dnp no)
+		(fields_autoplaced yes)
+		(property "Reference" "C55"
+			(at 381 226.06 90)
+			(effects
+				(font
+					(size 1.27 1.27)
+				)
+			)
+		)
+		(property "Value" "100nF"
+			(at 381 228.6 90)
+			(effects
+				(font
+					(size 1.27 1.27)
+				)
+			)
+		)
+		(property "Footprint" "Capacitor_SMD:C_0603_1608Metric"
+			(at 381 222.25 0)
+			(effects
+				(font
+					(size 1.27 1.27)
+				)
+				(hide yes)
+			)
+		)
+		(property "Datasheet" ""
+			(at 381 222.25 0)
+			(effects
+				(font
+					(size 1.27 1.27)
+				)
+				(hide yes)
+			)
+		)
+		(property "Description" ""
+			(at 381 222.25 0)
+			(effects
+				(font
+					(size 1.27 1.27)
+				)
+			)
+		)
+		(pin "1"
+		)
+		(pin "2"
+		)
+		(instances
+			(project "Radar1"
+				(path "/813c6d5a-f49c-4157-a259-eb6b4a93e133"
+					(reference "C55")
+					(unit 1)
+				)
+			)
+		)
+	)	(sheet_instances
 		(path "/"
 			(page "1")
 		)
 	)
+	(global_label "+1V8"
+		(shape input)
+		(at 378.46 222.25 90)
+		(effects
+			(font
+				(size 1.27 1.27)
+			)
+		)
+	)
+	(global_label "GND"
+		(shape input)
+		(at 383.54 222.25 90)
+		(effects
+			(font
+				(size 1.27 1.27)
+			)
+		)
+	)
