File: Radar1.kicad_sch (KiCad schematic)
At the start: 99 parts, among them J1 USB4215-03-A, J2 Barrel_Jack, J3 SMA-2.92mm-EndLaunch, J4 SMA-2.92mm-EndLaunch, U1 BGT24LTR11N16, U10 93LC56B-I/SN, U11 445I23D12M00000, U12 AMM-8211PSM, U13 TPS7A4700RGWT, U14 TPS7A2033PDBVR, U15 TPD2E009DBZR, U16 REF5025AID, U2 ADF4159WCCPZ, U3 OPA1656ID, U4 TPS7A2033PDBVR, U5 TPS7A2018PDBVR, U6 TPS7A4700RGWT, U7 FT2232HL-REEL, U8 ADS8353IPW, U9 ADP5600ACPZ-R7, Y1 ECS-TXO-2520MV-500-AN-TR

Commit message: Rev-E: PLL loop filter redesign — topology fix + computed values
The captured loop filter was an all-shunt RC ladder: a current-driven
ladder has no finite zero at V_TUNE, making the type-2 loop
unconditionally unstable (verified by exact network analysis, see
tools/pll_loop_filter.py). R4's input moves from the R3/C18 junction to
CPOUT, restoring the standard 3rd-order passive topology.

Values from BGT24LTR11 DS (Kvco 720M/2G Hz/V, VTUNE 0.7-2.5V, /16) and
ADF4159 (RSET 5.1k, Icp 2.5mA, fPFD 50MHz, N=483):
C17 910pF, R3 270R, C18 15nF, R4 560R, C19 270pF
-> fc 146 kHz, PM 52 deg (typ); all corners in docs/PLL-LOOP-FILTER.md.

Schematic: R4.1 global label LF_B->LF_A + 5 values (netlist regression:
exactly that delta). Board: R4.1 pad re-netted, LF_A/LF_B ripped and
rerouted, stale-geometry clearance/crossing defects from earlier heals
fixed (0 shorts / 0 clearance / 0 crossings). Routing backlog now 6 nets.

Co-Authored-By: Claude Fable 5 <noreply@anthropic.com>
Parts:
- C17: value 1nF -> 910pF
- C18: value 10nF -> 15nF
- C19: value 470pF -> 270pF
- R3: value 10k -> 270R
- R4: value 2.2k -> 560R
Connections:
- net LF_A: now also R4.1
- net LF_B: no longer R4.1
Changed lines of the file:
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@@
 		)
 	)
-	(global_label "LF_B"
+	(global_label "LF_A"
 		(shape input)
 		(at 309.88 166.37 180)
@@
 			)
 		)
-		(property "Value" "470pF"
+		(property "Value" "270pF"
 			(at 316.23 153.543 90)
 			(effects
@@
 			)
 		)
-		(property "Value" "10k"
+		(property "Value" "270R"
 			(at 316.23 184.15 90)
 			(effects
@@
 			)
 		)
-		(property "Value" "2.2k"
+		(property "Value" "560R"
 			(at 316.23 163.83 90)
 			(effects
@@
 			)
 		)
-		(property "Value" "10nF"
+		(property "Value" "15nF"
 			(at 316.23 173.863 90)
 			(effects
@@
 			)
 		)
-		(property "Value" "1nF"
+		(property "Value" "910pF"
 			(at 316.23 194.183 90)
 			(effects
